Commit message: attempt to fix arm urdf

File: doris_arm_description/urdf/doris_arm_description.urdf.xacro (robot description, xacro)
@@ -8,6 +8,6 @@
     <inertial>
       <origin xyz="0.0032335 -3.6289E-06 0.02346" rpy="0 0 0" />
-      <mass value="0.086496" />
-      <inertia ixx="0.002" ixy="0.0" ixz="0.0" iyy="0.002" iyz="0.0" izz="0.002" />
+      <mass value="0.001"/>
+        <inertia ixx="0.001" ixy="0" ixz="0" iyy="0.001" iyz="0" izz="0.001"/>
     </inertial>
     <visual>
@@ -30,6 +30,6 @@
     <inertial>
       <origin xyz="1.80019426116503E-06 0.0469908207821207 1.02798098779305E-05" rpy="0 0 0" />
-      <mass value="0.187371975468428" />
-      <inertia ixx="0.002" ixy="0.0" ixz="0.0" iyy="0.002" iyz="0.0" izz="0.002" />
+      <mass value="0.000187371975468428" />
+      <inertia ixx="0.001" ixy="0.0" ixz="0.0" iyy="0.001" iyz="0.0" izz="0.001" />
     </inertial>
     <visual>
@@ -60,6 +60,6 @@
     <inertial>
       <origin xyz="-1.08638707938674E-05 0.145957509942709 0.00428434606455026" rpy="0 0 0" />
-      <mass value="0.0731491894717436" />
-      <inertia ixx="0.002" ixy="0.0" ixz="0.0" iyy="0.002" iyz="0.0" izz="0.002" />
+      <mass value="0.001"/>
+        <inertia ixx="0.001" ixy="0" ixz="0" iyy="0.001" iyz="0" izz="0.001"/>
     </inertial>
     <visual>
@@ -90,6 +90,6 @@
     <inertial>
       <origin xyz="-3.11104449999267E-05 -0.0168263295023695 0.000457294178247414" rpy="0 0 0" />
-      <mass value="0.0892046248471317" />
-            <inertia ixx="0.002" ixy="0.0" ixz="0.0" iyy="0.002" iyz="0.0" izz="0.002" />
+      <mass value="0.001"/>
+        <inertia ixx="0.001" ixy="0" ixz="0" iyy="0.001" iyz="0" izz="0.001"/>
     </inertial>
     <visual>
@@ -120,6 +120,6 @@
     <inertial>
       <origin xyz="1.19120197594746E-08 -0.010083697233814 -0.0945595691856148" rpy="0 0 0" />
-      <mass value="0.108644948048519" />
-            <inertia ixx="0.002" ixy="0.0" ixz="0.0" iyy="0.002" iyz="0.0" izz="0.002" />
+      <mass value="0.001"/>
+        <inertia ixx="0.001" ixy="0" ixz="0" iyy="0.001" iyz="0" izz="0.001"/>
     </inertial>
     <visual>
@@ -150,6 +150,6 @@
     <inertial>
       <origin xyz="4.05516357848967E-05 -0.0160211563366842 -0.000189877443412478" rpy="0 0 0" />
-      <mass value="0.0768058991199202" />
-            <inertia ixx="0.002" ixy="0.0" ixz="0.0" iyy="0.002" iyz="0.0" izz="0.002" />
+      <mass value="0.001"/>
+        <inertia ixx="0.001" ixy="0" ixz="0" iyy="0.001" iyz="0" izz="0.001"/>
     </inertial>
     <visual>
@@ -180,6 +180,6 @@
     <inertial>
       <origin xyz="3.30999898656703E-07 -0.0146248804164249 0.0456383476057014" rpy="0 0 0" />
-      <mass value="0.15161780969895" />
-            <inertia ixx="0.002" ixy="0.0" ixz="0.0" iyy="0.002" iyz="0.0" izz="0.002" />
+      <mass value="0.001"/>
+        <inertia ixx="0.001" ixy="0" ixz="0" iyy="0.001" iyz="0" izz="0.001"/>
     </inertial>
     <visual>
@@ -210,6 +210,6 @@
     <inertial>
       <origin xyz="0.0230127657229507 0.000126473527769386 0.00158449770655011" rpy="0 0 0" />
-      <mass value="0.0174078384350788" />
-            <inertia ixx="0.002" ixy="0.0" ixz="0.0" iyy="0.002" iyz="0.0" izz="0.002" />
+      <mass value="0.001"/>
+        <inertia ixx="0.001" ixy="0" ixz="0" iyy="0.001" iyz="0" izz="0.001"/>
     </inertial>
     <visual>
@@ -238,6 +238,6 @@
     <inertial>
       <origin xyz="-2.5501E-07 -0.0020883 0.03999" rpy="0 0 0" />
-      <mass value="0.0083226" />
-            <inertia ixx="0.002" ixy="0.0" ixz="0.0" iyy="0.002" iyz="0.0" izz="0.002" />
+      <mass value="0.001"/>
+        <inertia ixx="0.001" ixy="0" ixz="0" iyy="0.001" iyz="0" izz="0.001"/>
     </inertial>
     <visual>
@@ -268,6 +268,6 @@
     <inertial>
       <origin xyz="-2.55484871550249E-07 0.0123652457374703 0.0380876079681996" rpy="0 0 0" />
-      <mass value="0.00832263335631547" />
-            <inertia ixx="0.002" ixy="0.0" ixz="0.0" iyy="0.002" iyz="0.0" izz="0.002" />
+      <mass value="0.001"/>
+        <inertia ixx="0.001" ixy="0" ixz="0" iyy="0.001" iyz="0" izz="0.001"/>
     </inertial>
     <visual>
