Commit message: added kinect v2 to collsion and visual

File: doris_sensors_description/urdf/kinect_camera.urdf.xacro (robot description, xacro)
@@ -14,5 +14,5 @@
           <origin xyz="0 0 0" rpy="0 0 0" />
           <geometry>
-            <mesh filename="package://hector_sensors_description/meshes/kinect_camera/kinect_camera_simple.dae"/>
+            <mesh filename="package://doris_sensors_description/meshes/kinect_camera/sensors/kinectv2.stl"/>
           </geometry>
         </visual>
@@ -20,5 +20,5 @@
           <origin xyz="0 0 0" rpy="0 0 0" />
           <geometry>
-            <mesh filename="package://hector_sensors_description/meshes/kinect_camera/kinect_camera_simple.stl"/>
+            <mesh filename="package://doris_sensors_description/meshes/kinect_camera/sensors/kinectv2.stl"/>
           </geometry>
         </collision>
